Commit message: URDF modified for new end effector, d435 mounted it correct position with errors in rpy accounted for

File: urdf/panda_arm_suction_cam_new.urdf.xacro (robot description, xacro)
@@ -4,5 +4,5 @@
   <!-- Different xacro files for d435 and l515-->
   <xacro:include filename="$(find depth_enhance_robot)/urdf/suction_cup_d435.xacro"/>
-  <!-- <xacro:include filename="$(find depth_enhance_robot)/urdf/suction_cup_new.xacro"/> -->
+  <!-- <xacro:include filename="$(find depth_enhance_robot)/urdf/suction_cup_d435.xacro"/> -->
   <!--<xacro:include filename="$(find franka_description)/robots/hand.xacro"/>-->
   <!-- for simulation -->
@@ -13,5 +13,5 @@
   <!-- end for simulation -->
   <xacro:panda_arm />
-  <xacro:suction ns="panda" rpy="0 0 ${-pi/4}" connected_to="panda_link8"/>
+  <xacro:suction ns="panda" rpy="0 0 ${-pi/4}" xyz="0 0 0" connected_to="panda_link8"/>
   <!-- for simulation -->
   <xacro:arg name="robot_name" default="panda"/>

File: urdf/suction_cup_l515.xacro (robot description, xacro)
@@ -3,6 +3,6 @@
   <xacro:macro name="suction" params="connected_to:='' ns:='' rpy:='0 0 0' xyz:='0 0 0' ">
     <xacro:unless value="${connected_to == ''}">
-    <xacro:include filename="$(find realsense2_description)/urdf/_d435.urdf.xacro"/>
-    <!--<xacro:include filename="$(find realsense2_description)/urdf/_l515.urdf.xacro"/>-->
+    <!-- <xacro:include filename="$(find realsense2_description)/urdf/_d435.urdf.xacro"/> -->
+    <xacro:include filename="$(find realsense2_description)/urdf/_l515.urdf.xacro"/>
     <link name="${ns}_suction_rect"/>
       <joint name="${ns}_suction_joint" type="fixed">
@@ -72,15 +72,15 @@
 -->
 <link name="c_link" />
-<xacro:sensor_d435 parent="c_link">
+<xacro:sensor_l515 parent="c_link">
   <!--<origin xyz="0.01015 0.05 -0.0125" rpy="${pi/2} 0 0"/>-->
-  <!-- Camera sligthly tilted: Roll adjusted by 0.02 radians pitch adjusted by 0.025 radians -->
-  <origin xyz="0 0 0" rpy="${pi+0.02} ${-pi/2-0.025} 0"/>
+  <!-- Camera sligthly tilted: Roll adjusted by 0.015 radians - pitch adjusted by 0.025 radians -->
+  <origin xyz="0 0 0" rpy="${pi} ${-pi/2-0.025} 0"/>
 <!--<origin xyz="0.01015 0.05 -0.0125" rpy="${pi/2} 0 0"/> -->
-</xacro:sensor_d435>
+</xacro:sensor_l515>
 <joint name="basetocam" type="fixed">
   <parent link="shift_origin" />
   <child link="c_link" />
   <!--<origin rpy="0 ${-pi/2} ${-pi/2} " xyz="0.043 -0.01265 0.004"/>-->
-  <origin rpy="0 0 0 " xyz="${0.02-0.0125} 0 0.0125"/>
+  <origin rpy="0.025 0 0 " xyz="${0.02-0.0125} 0 0.0125"/>
   <!--<origin rpy="3.141593 -1.571 0 " xyz="0 0 0"/>
   <origin rpy="3.1415 -1.571 0 " xyz="0.040 -0.0175 0.066"/>-->

Commit message: A URDF model that works by rotating joint6 by 3 degrees

File: urdf/panda_arm_suction_cam_new.urdf.xacro (robot description, xacro)
@@ -3,5 +3,5 @@
   <xacro:include filename="$(find franka_description)/robots/panda_arm.xacro"/>
   <!-- Different xacro files for d435 and l515-->
-  <xacro:include filename="$(find depth_enhance_robot)/urdf/suction_cup_d435.xacro"/>
+  <xacro:include filename="$(find depth_enhance_robot)/urdf/suction_cup_l515.xacro"/>
   <!-- <xacro:include filename="$(find depth_enhance_robot)/urdf/suction_cup_d435.xacro"/> -->
   <!--<xacro:include filename="$(find franka_description)/robots/hand.xacro"/>-->

File: urdf/suction_cup_l515.xacro (robot description, xacro)
@@ -16,4 +16,5 @@
       <parent link="${connected_to}"/>
       <child link="${ns}_suction_rect"/>
+      <!-- pitch to account for end effector angle -->
       <origin xyz="0 0 0" rpy="0 0 ${-pi/4}"/>
       <!--<origin xyz="0 0 0" rpy="0 0 ${-pi/4}"/>-->
@@ -29,5 +30,5 @@
  <origin xyz="0 0 0" rpy="${-pi/2} 0 ${-pi/2}"/>
   <geometry>
-    <mesh filename="package://depth_enhance_robot/urdf/stykkibody.STL"
+    <mesh filename="package://depth_enhance_robot/urdf/stykkibodyV3.STL"
     scale="0.001 0.001 0.001"/>
   </geometry>
@@ -36,5 +37,5 @@
 <origin xyz="0 0 0" rpy="${-pi/2} 0 ${-pi/2}"/>
   <geometry>
-    <mesh filename="package://depth_enhance_robot/urdf/stykkibody.STL"
+    <mesh filename="package://depth_enhance_robot/urdf/stykkibodyV3.STL"
     scale="0.001 0.001 0.001"/>
   </geometry>
@@ -50,5 +51,5 @@
   <parent link="${ns}_suction_rect"/>
   <child link="${ns}_suction_end"/>
-  <origin xyz="0 0 0.139" rpy="0 0 0"/>
+  <origin xyz="0 0 0.222" rpy="0 0 0"/>
 </joint>
 <link name="shift_origin"/>
@@ -57,5 +58,5 @@
   <child link="shift_origin"/>
   <!-- <origin xyz="0.032 0 0.004 " rpy="0 0 0 "/> -->
-  <origin xyz="0.032 0 0.002 " rpy="0 0 0 "/>
+  <origin xyz="0.04 0 0.004 " rpy="0 0 0 "/>
 </joint>
 <link name="picking_camera_link"/>
@@ -70,20 +71,29 @@
 x er i att ad i att ad vegg ef hann er i upphafsstodu
 y er i att ad tokkum
+Calibration: RPY -> 0.0392, 0.0329, 0.0262
 -->
-<link name="c_link" />
+<!-- <link name="c_link"/>
 <xacro:sensor_l515 parent="c_link">
-  <!--<origin xyz="0.01015 0.05 -0.0125" rpy="${pi/2} 0 0"/>-->
-  <!-- Camera sligthly tilted: Roll adjusted by 0.015 radians - pitch adjusted by 0.025 radians -->
-  <origin xyz="0 0 0" rpy="${pi} ${-pi/2-0.025} 0"/>
-<!--<origin xyz="0.01015 0.05 -0.0125" rpy="${pi/2} 0 0"/> -->
+  <origin xyz="-0.030325 0 0.013" rpy="${pi} ${-pi/2-0.01} 0"/>
+</xacro:sensor_l515> -->
+<!-- <joint name="basetocam" type="fixed">
+  <parent link="shift_origin" />
+  <child link="c_link" />
+  #<origin rpy="0.025 0 0 " xyz="${0.02-0.0133} 0 0.0125"/>#
+  <origin rpy="0.021 0 0 " xyz="0.02 0 0"/>
+</joint> -->
+<link name="c_link"/>
+<xacro:sensor_l515 parent="c_link">
+  <!-- <origin xyz="${-0.030325+0.02} 0 0.013" rpy="${pi} ${-pi/2-0.01} 0"/> -->
+  <origin xyz="${-0.030325+0.02} 0 ${0.013+0.002}" rpy="${pi} ${-pi/2} 0"/>
 </xacro:sensor_l515>
 <joint name="basetocam" type="fixed">
   <parent link="shift_origin" />
   <child link="c_link" />
-  <!--<origin rpy="0 ${-pi/2} ${-pi/2} " xyz="0.043 -0.01265 0.004"/>-->
-  <origin rpy="0.025 0 0 " xyz="${0.02-0.0125} 0 0.0125"/>
-  <!--<origin rpy="3.141593 -1.571 0 " xyz="0 0 0"/>
-  <origin rpy="3.1415 -1.571 0 " xyz="0.040 -0.0175 0.066"/>-->
+  <!-- <origin rpy="0.025 0 0 " xyz="${0.02-0.0133} 0 0.0125"/> -->
+  <!-- <origin rpy="0.021 0 0 " xyz="0 0 0"/> -->
+  <origin rpy="0.02 0.04 0 " xyz="0 0 0"/>
 </joint>
+<!-- Roll: 0.03 gott - Pitch: 0.04-->
 <!--<joint name="kinect_joint" type="fixed">
     <parent link="${ns}_suction_cup" />

File: urdf/suction_cup_l515old.xacro (robot description, xacro)
@@ -3,6 +3,6 @@
   <xacro:macro name="suction" params="connected_to:='' ns:='' rpy:='0 0 0' xyz:='0 0 0' ">
     <xacro:unless value="${connected_to == ''}">
-    <xacro:include filename="$(find realsense2_description)/urdf/_d435.urdf.xacro"/>
-    <!--<xacro:include filename="$(find realsense2_description)/urdf/_l515.urdf.xacro"/>-->
+    <!-- <xacro:include filename="$(find realsense2_description)/urdf/_d435.urdf.xacro"/> -->
+    <xacro:include filename="$(find realsense2_description)/urdf/_l515.urdf.xacro"/>
     <link name="${ns}_suction_rect"/>
       <joint name="${ns}_suction_joint" type="fixed">
@@ -29,5 +29,5 @@
  <origin xyz="0 0 0" rpy="${-pi/2} 0 ${-pi/2}"/>
   <geometry>
-    <mesh filename="package://depth_enhance_robot/urdf/stykkibodyV3.STL"
+    <mesh filename="package://depth_enhance_robot/urdf/stykkibody.STL"
     scale="0.001 0.001 0.001"/>
   </geometry>
@@ -50,5 +50,5 @@
   <parent link="${ns}_suction_rect"/>
   <child link="${ns}_suction_end"/>
-  <origin xyz="0 0 0.21" rpy="0 0 0"/>
+  <origin xyz="0 0 0.22" rpy="0 0 0"/>
 </joint>
 <link name="shift_origin"/>
@@ -57,5 +57,5 @@
   <child link="shift_origin"/>
   <!-- <origin xyz="0.032 0 0.004 " rpy="0 0 0 "/> -->
-  <origin xyz="0.04 0 0.004 " rpy="0 0 0 "/>
+  <origin xyz="0.032 0 0.002 " rpy="0 0 0 "/>
 </joint>
 <link name="picking_camera_link"/>
@@ -72,16 +72,17 @@
 -->
 <link name="c_link" />
-<xacro:sensor_d435 parent="c_link">
+<xacro:sensor_l515 parent="c_link">
   <!--<origin xyz="0.01015 0.05 -0.0125" rpy="${pi/2} 0 0"/>-->
-  <!-- Camera sligthly tilted: Roll adjusted by 0.02 radians pitch adjusted by 0.025 radians -->
-  <!-- <origin xyz="0 0 0" rpy="${pi+0.02} ${-pi/2-0.025} 0"/> -->
-  <origin xyz="-0.0125 0 ${0.0125-0.002}" rpy="${pi} ${-pi/2} 0"/>
-</xacro:sensor_d435>
-<!-- Roll adjusted here since roll seems to control yaw for the d435 xacro sensor -->
+  <!-- Camera sligthly tilted: Roll adjusted by 0.015 radians - pitch adjusted by 0.025 radians -->
+  <origin xyz="0 0 0" rpy="${pi} ${-pi/2-0.025} 0"/>
+<!--<origin xyz="0.01015 0.05 -0.0125" rpy="${pi/2} 0 0"/> -->
+</xacro:sensor_l515>
 <joint name="basetocam" type="fixed">
-  <parent link="shift_origin"/>
+  <parent link="shift_origin" />
   <child link="c_link" />
-  <!-- <origin rpy="0.02 -0.045 0 " xyz="0.02 0 0"/> -->
-  <origin rpy="0.05 -0.01 0 " xyz="0.02 0 0"/>
+  <!--<origin rpy="0 ${-pi/2} ${-pi/2} " xyz="0.043 -0.01265 0.004"/>-->
+  <origin rpy="0.025 0 0 " xyz="${0.02-0.0125} 0 0.0125"/>
+  <!--<origin rpy="3.141593 -1.571 0 " xyz="0 0 0"/>
+  <origin rpy="3.1415 -1.571 0 " xyz="0.040 -0.0175 0.066"/>-->
 </joint>
 <!--<joint name="kinect_joint" type="fixed">

Commit message: d435 URDF model corrected

File: urdf/panda_arm_suction_cam_new.urdf.xacro (robot description, xacro)
@@ -3,5 +3,5 @@
   <xacro:include filename="$(find franka_description)/robots/panda_arm.xacro"/>
   <!-- Different xacro files for d435 and l515-->
-  <xacro:include filename="$(find depth_enhance_robot)/urdf/suction_cup_l515.xacro"/>
+  <xacro:include filename="$(find depth_enhance_robot)/urdf/suction_cup_d435.xacro"/>
   <!-- <xacro:include filename="$(find depth_enhance_robot)/urdf/suction_cup_d435.xacro"/> -->
   <!--<xacro:include filename="$(find franka_description)/robots/hand.xacro"/>-->

File: urdf/suction_cup_d435.xacro (robot description, xacro)
@@ -50,5 +50,5 @@
   <parent link="${ns}_suction_rect"/>
   <child link="${ns}_suction_end"/>
-  <origin xyz="0 0 0.21" rpy="0 0 0"/>
+  <origin xyz="0 0 0.222" rpy="0 0 0"/>
 </joint>
 <link name="shift_origin"/>
@@ -83,6 +83,8 @@
   <child link="c_link" />
   <!-- <origin rpy="0.02 -0.045 0 " xyz="0.02 0 0"/> -->
-  <origin rpy="0.05 -0.01 0 " xyz="0.02 0 0"/>
+  <origin rpy="0.026 -0.01 0 " xyz="0.02 0 0"/>
+  <!-- <origin rpy="0 0 0 " xyz="0.02 0 0"/> -->
 </joint>
+<!-- R: 0.28 acceptable -->
 <!--<joint name="kinect_joint" type="fixed">
     <parent link="${ns}_suction_cup" />

File: urdf/suction_cup_l515.xacro (robot description, xacro)
@@ -93,5 +93,6 @@
   <!-- <origin rpy="0.025 0 0 " xyz="${0.02-0.0133} 0 0.0125"/> -->
   <!-- <origin rpy="0.021 0 0 " xyz="0 0 0"/> -->
-  <origin rpy="0.02 0.04 0 " xyz="0 0 0"/>
+  <!-- <origin rpy="0.02 0.04 0 " xyz="0 0 0"/> Settings that worked with joint6 adjusted -->
+  <origin rpy="0 0 0 " xyz="0 0 0"/>
 </joint>
 <!-- Roll: 0.03 gott - Pitch: 0.04-->
