Commit message: Changed initial position, a lot of tests and functions added to picktestand the data gathering algorithm is a work in progress

File: urdf/suction_cup_d435.xacro (robot description, xacro)
@@ -83,6 +83,6 @@
   <child link="c_link" />
   <!-- <origin rpy="0.02 -0.045 0 " xyz="0.02 0 0"/> -->
-  <origin rpy="0.026 -0.01 0 " xyz="0.02 0 0"/>
-  <!-- <origin rpy="0 0 0 " xyz="0.02 0 0"/> -->
+  <!-- <origin rpy="0.026 -0.01 0 " xyz="0.02 0 0"/> -->
+  <origin rpy="0 0 0 " xyz="0.02 0 0"/>
 </joint>
 <!-- R: 0.28 acceptable -->
